File: plant_waterer/plant_waterer.kicad_sch (KiCad schematic)
At the start: 30 parts, among them J2 Conn_01x02, J3 PJ-002AH, J4 Conn_01x03, U1 ZXBM5210-SP-13, U2 OLED_DISP, U4 ESD7002, U5 AP2204R-5.0TRG1, U6 PicoW

Commit message: Cleanup for V5
Parts:
- added C1: 22nF, Capacitor_SMD:C_0805_2012Metric_Pad1.18x1.45mm_HandSolder, symbol Device:C
- added L1: 100uH, Inductor_SMD:L_0805_2012Metric_Pad1.05x1.20mm_HandSolder, symbol Device:L
- added R1: 100, Resistor_SMD:R_0805_2012Metric_Pad1.20x1.40mm_HandSolder, symbol Device:R
- U4: footprint Package_TO_SOT_SMD:SOT-323_SC-70_Handsoldering -> Package_TO_SOT_SMD:SOT-323_SC-70
- renumbered C7 to C2, C1 to C3, C2 to C4, C3 to C5, C4 to C6, C5 to C7, C6 to C8, J2 to J1, J3 to J2, J4 to J3, R1 to R5, TP4 to TP1, TP1 to TP2, TP2 to TP3, TP3 to TP4, U6 to U1, U1 to U2, U2 to U3
Connections:
- net GND: now also C1.1
- net SCL: now also U1.17 (GPIO13), U4.2; no longer U1.32 (GPIO27_ADC1), U4.1
- net SDA: now also U1.16 (GPIO12), U4.1, R1.1; no longer U1.31 (GPIO26_ADC0), U4.2
- new net: C1.2, L1.2, U1.31 (GPIO26_ADC0)
- new net: L1.1, R1.2
Other:
- note added: "NOPOP if PWM"
- note added: "NOPOP if not PWM"
- note added: "PWM Low Pass Filter"
- moved on the sheet: D2, J3, JP1, R2, R3, R4, R5, RV1, TP1, TP5, U1, U3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
