File: plant_combined/plant_combined/plant_combined.kicad_sch (KiCad schematic)
At the start: 37 parts, among them J2 PJ-002AH, J3 Conn_01x02, U10 ZXBM5210-SP-13, U2 OLED_DISP, U8 PicoW, U9 AP62200WU-7

Commit message: Fixes for footprints
Parts:
- removed 5V: TestPoint, TestPoint:TestPoint_Loop_D1.80mm_Drill1.0mm_Beaded, symbol Connector:TestPoint
- removed D2: BZX84C15T, Package_TO_SOT_SMD:SOT-23, symbol Diode:BZX84Cxx
- added D5: BZX84Cxx, Package_TO_SOT_SMD:SOT-523, symbol MySymbols:BZX84Cxx
- added TP7: TestPoint, Library:TestPoint_2Pads_Pitch2.54mm_Drill1mm, symbol Connector:TestPoint_2Pole
- SCL1: renamed from SCL; footprint TestPoint:TestPoint_2Pads_Pitch5.08mm_Drill1.3mm -> Library:TestPoint_2Pads_Pitch2.54mm_Drill1mm
- SDA1: renamed from SDA; footprint TestPoint:TestPoint_2Pads_Pitch5.08mm_Drill1.3mm -> Library:TestPoint_2Pads_Pitch2.54mm_Drill1mm
- renumbered 12V to TP2
Connections:
- net +12P: now also D5.3 (K)
- net +5V: now also TP7.2
- net GND: now also TP7.1
- net at C2.1, D3.3 (G), R3.2: now also D5.1 (A)
Other:
- moved on the sheet: C15, C2, C8, D1, D3, R3
