File: plant_combined/plant_combined/tdr_sensor.kicad_sch (KiCad schematic)
At the start: 31 parts, among them J1 SMA-J-P-H-ST-EM1, U1 SI5351A-B-GT, U3 TDC7200PWR, U4 ADCMP600BKSZ-R2, U5 74AC14SC, U6 ESD7002, U7 MCP1700T, Y1 Crystal_GND24

Commit message: Fixes for footprints
Parts:
- removed MOSI, SCLK: TestPoint, TestPoint:TestPoint_Loop_D1.80mm_Drill1.0mm_Beaded, symbol Connector:TestPoint
- added MOSI1, SCLK1: TestPoint, Library:TestPoint_2Pads_Pitch2.54mm_Drill1mm, symbol Connector:TestPoint_2Pole
- added TP10: TestPoint_2Pole, Library:TestPoint_2Pads_Pitch2.54mm_Drill1mm, symbol Connector:TestPoint_2Pole
- TP7: footprint TestPoint:TestPoint_2Pads_Pitch5.08mm_Drill1.3mm -> Library:TestPoint_2Pads_Pitch2.54mm_Drill1mm
- V REF1: renamed from V REF
- renumbered CLK to CLK1, START to START1, STOP to STOP1
Connections:
- net +3.3VA: now also TP10.2
- net GND: now also MOSI1.2, SCLK1.2, TP10.1
- net MOSI: now also MOSI1.1
- net SCLK: now also SCLK1.1
- no-connect marks 0 -> 1
